File: coleco-adam-ade-pro-shield.sch (KiCad schematic (older format))
At the start: 26 parts, among them J1 RJ12, P1 Digital, P2 Power, P3 Analog, P4 Analog, P5 PWM, P6 PWM, P7 Communication, Q1 2N3906, SW1 SWAP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

Commit message: Add some docs
Parts:
- C1: Comment (none) -> Optional
- JP1, P1, P2, P3, P4, P5, P6, P7: Comment (none) -> Use 2.54mm male headers
- R3: Comment (none) -> Activity LED brightness
- R4: Comment (none) -> LCD backlighting brightness
- RV1: footprint Potentiometer_THT:Potentiometer_Bourns_3296W_Vertical -> 3362P-1-103:TRIM_3362P-1-103
- SW1, SW2, SW3, SW4, SW5, SW6, SW7: Comment (none) -> Standard 6x6mm tactical switch
Changed lines of the file:
@@
 encoding utf-8
 Sheet 1 1
-Title ""
-Date "mar. 31 mars 2015"
-Rev ""
+Title "Coleco Adam ADE Pro Shield"
+Date "2021-03-05"
+Rev "v1.0"
 Comp ""
 Comment1 ""
@@
 F 2 "Socket_Arduino_Mega:Socket_Strip_Arduino_1x08" H 9550 1650 50  0001 C CNN
 F 3 "" H 9550 1650 50  0000 C CNN
+F 4 "Use 2.54mm male headers" H 9550 1650 50  0001 C CNN "Comment"
 	1    9550 1650
 	1    0    0    -1
@@
 F 2 "Socket_Arduino_Mega:Socket_Strip_Arduino_1x10" H 9950 1550 50  0001 C CNN
 F 3 "" H 9950 1550 50  0000 C CNN
+F 4 "Use 2.54mm male headers" H 9950 1550 50  0001 C CNN "Comment"
 	1    9950 1550
 	-1   0    0    -1
@@
 F 2 "Socket_Arduino_Mega:Socket_Strip_Arduino_1x08" H 9550 2750 50  0001 C CNN
 F 3 "" H 9550 2750 50  0000 C CNN
+F 4 "Use 2.54mm male headers" H 9550 2750 50  0001 C CNN "Comment"
 	1    9550 2750
 	1    0    0    -1
@@
 F 2 "Socket_Arduino_Mega:Socket_Strip_Arduino_1x08" H 9950 2750 50  0001 C CNN
 F 3 "" H 9950 2750 50  0000 C CNN
+F 4 "Use 2.54mm male headers" H 9950 2750 50  0001 C CNN "Comment"
 	1    9950 2750
 	-1   0    0    -1
@@
 F 2 "Socket_Arduino_Mega:Socket_Strip_Arduino_1x08" H 9550 3700 50  0001 C CNN
 F 3 "" H 9550 3700 50  0000 C CNN
+F 4 "Use 2.54mm male headers" H 9550 3700 50  0001 C CNN "Comment"
 	1    9550 3700
 	1    0    0    -1
@@
 F 2 "Socket_Arduino_Mega:Socket_Strip_Arduino_1x08" H 9950 3700 50  0001 C CNN
 F 3 "" H 9950 3700 50  0000 C CNN
+F 4 "Use 2.54mm male headers" H 9950 3700 50  0001 C CNN "Comment"
 	1    9950 3700
 	-1   0    0    -1
@@
 F 2 "Socket_Arduino_Mega:Socket_Strip_Arduino_2x18" H 9700 4000 50  0001 C CNN
 F 3 "" H 9700 4000 50  0000 C CNN
+F 4 "Use 2.54mm male headers" H 9700 5050 50  0001 C CNN "Comment"
 	1    9700 5050
 	0    -1   1    0
@@
 F 2 "Button_Switch_THT:SW_TH_Tactile_Omron_B3F-10xx" H 6800 3500 50  0001 C CNN
 F 3 "http://www.apem.com/int/index.php?controller=attachment&id_attachment=1371" H 6800 3500 50  0001 C CNN
+F 4 "Standard 6x6mm tactical switch" H 6800 3200 50  0001 C CNN "Comment"
 	1    6800 3200
 	1    0    0    -1
@@
 F 2 "Button_Switch_THT:SW_TH_Tactile_Omron_B3F-10xx" H 6800 3950 50  0001 C CNN
 F 3 "http://www.apem.com/int/index.php?controller=attachment&id_attachment=1371" H 6800 3950 50  0001 C CNN
+F 4 "Standard 6x6mm tactical switch" H 6800 3650 50  0001 C CNN "Comment"
 	1    6800 3650
 	1    0    0    -1
@@
 F 2 "Button_Switch_THT:SW_TH_Tactile_Omron_B3F-10xx" H 6800 4400 50  0001 C CNN
 F 3 "http://www.apem.com/int/index.php?controller=attachment&id_attachment=1371" H 6800 4400 50  0001 C CNN
+F 4 "Standard 6x6mm tactical switch" H 6800 4100 50  0001 C CNN "Comment"
 	1    6800 4100
 	1    0    0    -1
@@
 F 2 "Button_Switch_THT:SW_TH_Tactile_Omron_B3F-10xx" H 6800 4850 50  0001 C CNN
 F 3 "http://www.apem.com/int/index.php?controller=attachment&id_attachment=1371" H 6800 4850 50  0001 C CNN
+F 4 "Standard 6x6mm tactical switch" H 6800 4550 50  0001 C CNN "Comment"
 	1    6800 4550
 	1    0    0    -1
@@
 F 2 "Button_Switch_THT:SW_TH_Tactile_Omron_B3F-10xx" H 6800 5300 50  0001 C CNN
 F 3 "http://www.apem.com/int/index.php?controller=attachment&id_attachment=1371" H 6800 5300 50  0001 C CNN
+F 4 "Standard 6x6mm tactical switch" H 6800 5000 50  0001 C CNN "Comment"
 	1    6800 5000
 	1    0    0    -1
@@
 F 2 "Button_Switch_THT:SW_TH_Tactile_Omron_B3F-10xx" H 6800 6250 50  0001 C CNN
 F 3 "http://www.apem.com/int/index.php?controller=attachment&id_attachment=1371" H 6800 6250 50  0001 C CNN
+F 4 "Standard 6x6mm tactical switch" H 6800 5950 50  0001 C CNN "Comment"
 	1    6800 5950
 	1    0    0    -1
@@
 F 2 "Button_Switch_THT:SW_TH_Tactile_Omron_B3F-10xx" H 6800 5750 50  0001 C CNN
 F 3 "http://www.apem.com/int/index.php?controller=attachment&id_attachment=1371" H 6800 5750 50  0001 C CNN
+F 4 "Standard 6x6mm tactical switch" H 6800 5450 50  0001 C CNN "Comment"
 	1    6800 5450
 	1    0    0    -1
@@
 F 0 "RV1" H 7482 954 50  0000 R CNN
 F 1 "R_POT_TRIM_US" H 7482 1045 50  0000 R CNN
-F 2 "Potentiometer_THT:Potentiometer_Bourns_3296W_Vertical" H 7550 1000 50  0001 C CNN
+F 2 "3362P-1-103:TRIM_3362P-1-103" H 7550 1000 50  0001 C CNN
 F 3 "~" H 7550 1000 50  0001 C CNN
 	1    7550 1000
@@
 F 2 "Resistor_THT:R_Axial_DIN0207_L6.3mm_D2.5mm_P7.62mm_Horizontal" V 7280 1300 50  0001 C CNN
 F 3 "~" H 7350 1300 50  0001 C CNN
+F 4 "LCD backlighting brightness" H 7350 1300 50  0001 C CNN "Comment"
 	1    7350 1300
 	0    1    1    0
@@
 F 2 "Resistor_THT:R_Axial_DIN0207_L6.3mm_D2.5mm_P7.62mm_Horizontal" V 4830 3850 50  0001 C CNN
 F 3 "~" H 4900 3850 50  0001 C CNN
+F 4 "Activity LED brightness" H 4900 3850 50  0001 C CNN "Comment"
 	1    4900 3850
 	0    1    1    0
@@
 F 2 "Connector_PinHeader_2.54mm:PinHeader_2x01_P2.54mm_Vertical" H 4300 4350 50  0001 C CNN
 F 3 "~" H 4300 4350 50  0001 C CNN
+F 4 "Use 2.54mm male headers" H 4300 4350 50  0001 C CNN "Comment"
 	1    4300 4350
 	1    0    0    -1
@@
 F 2 "Capacitor_THT:CP_Radial_D4.0mm_P1.50mm" H 4600 4500 50  0001 C CNN
 F 3 "~" H 4600 4500 50  0001 C CNN
+F 4 "Optional" H 4600 4500 50  0001 C CNN "Comment"
 	1    4600 4500
 	1    0    0    -1
